Commit message: hand_urdf_test

File: assets/robots/inspire_rh56/inspire_rh56_right.urdf (robot description, URDF)
Before this commit: robot inspire_rh56_right, 20 links, 19 joints
Links:
- link middle_proximal: geometry collision mesh filename=meshes/collision/right_index_proximal.obj; visual mesh filename=meshes/visual/right_middle_proximal.glb
